File: EXP/GPU_SCH/main.kicad_sch (KiCad schematic)
At the start: 66 parts, among them J1 Conn_02x10_Counter_Clockwise, J2 Conn_01x03, J6 DB15_Female_HighDensity, Q1 FDV301N, Q2 FDV301N, Q3 FDV301N, U1 74HC4040, U10 74LS157, U11 74HC688, U12 74HC688, U13 74LS157, U14 74LS157, U15 74HC688, U16 74HC688, U17 74LS157, U18 74HC373, U19 74HC373, U2 74HC74, U20 74HC373, U21 74LS20, U22 74LS151, U23 74HC373, U24 74HC74, U25 74HC00, U3 74HC14, U4 74HC4040, U5 IS6xC1024AL-xxT, U6 74HC238, U7 74HC688, U8 74HC688, U9 74HC373, Y2 CXO_DIP8

Commit message: Add files via upload
Parts:
- J6: footprint Connector_Dsub:DSUB-15-HD_Pins_Horizontal_P2.29x1.90mm_EdgePinOffset3.03mm_Housed_MountingHolesOffset4.94mm -> Connector_Dsub:DSUB-15-HD_Socket_Horizontal_P2.29x1.90mm_EdgePinOffset3.03mm_Housed_MountingHolesOffset4.94mm
Connections:
- net +5V: no longer U25.1
- net A0: now also U6.1 (A0)
- net A1: now also U6.2 (A1)
- net A16: now also U25.8; no longer U25.11
- net F_EDIT: now also U25.5; no longer U25.9
- net F_OUT: now also U25.2; no longer U25.5
- net PRE: now also U25.1
- net VCLK: now also U3.13
- net X2: now also U25.12, U25.13; no longer U3.13
- net ~{PRE}: now also U25.4; no longer U25.10, U25.2
- net ~{VCLK}: now also U3.12
- net at U25.6: now also U25.10; no longer U25.12
- net at U21.4: now also U25.11; no longer U3.12
- net at U25.3: now also U25.9; no longer U25.4
Other:
- moved on the sheet: U21A, U25A, U25B, U25C, U25D, U3D, U3E, U3F
